File: powerBlock/_autosave-powerBlock.sch (KiCad schematic (older format))
At the start: 30 parts, among them Q1 Q_PNP_EBC, Q2 Q_PNP_EBC, Q3 Q_PNP_EBC, U1 STM32F030C8Tx, U2 74HC164, U3 74HC164, U4 BA56-12SRWA

Commit message: Добавил индикаторную панель. Подключил диод
Connections:
- net GND: now also D1.1 (K), D2.1 (K), D3.1 (K), D4.1 (K), D5.1 (K), D7.1 (K), D8.1 (K), U2.7 (GND)
Changed lines of the file:
@@
 SWDIO
 $Comp
-L power:+5V #PWR?
+L power:+5V #PWR0105
 U 1 1 5E93BF1A
 P 1350 5650
-F 0 "#PWR?" H 1350 5500 50  0001 C CNN
+F 0 "#PWR0105" H 1350 5500 50  0001 C CNN
 F 1 "+5V" H 1365 5823 50  0000 C CNN
 F 2 "" H 1350 5650 50  0001 C CNN
@@
 $EndComp
 $Comp
-L power:GND #PWR?
+L power:GND #PWR0106
 U 1 1 5E940E3D
 P 8650 2900
-F 0 "#PWR?" H 8650 2650 50  0001 C CNN
+F 0 "#PWR0106" H 8650 2650 50  0001 C CNN
 F 1 "GND" H 8655 2727 50  0000 C CNN
 F 2 "" H 8650 2900 50  0001 C CNN
@@
 	-1   0    0    1
 $EndComp
-Wire Wire Line
-	7400 2400 8100 2400
 $Comp
 L Device:LED D7
@@
 	7400 2600 8100 2600
 NoConn ~ 6500 2800
+Wire Wire Line
+	8000 2700 8650 2700
+Wire Wire Line
+	8650 2700 8650 2900
+Wire Wire Line
+	8650 2700 8650 2600
+Wire Wire Line
+	8650 2600 8400 2600
+Connection ~ 8650 2700
+Wire Wire Line
+	8650 2600 8650 2500
+Wire Wire Line
+	8650 2500 8000 2500
+Connection ~ 8650 2600
+Wire Wire Line
+	8650 2400 8650 2500
+Connection ~ 8650 2500
+Wire Wire Line
+	8400 2400 8650 2400
+Wire Wire Line
+	7400 2400 8100 2400
+Wire Wire Line
+	8000 2300 8650 2300
+Wire Wire Line
+	8650 2300 8650 2400
+Connection ~ 8650 2400
+Wire Wire Line
+	8650 2300 8650 2200
+Wire Wire Line
+	8650 2200 8400 2200
+Connection ~ 8650 2300
+Wire Wire Line
+	8000 2100 8650 2100
+Wire Wire Line
+	8650 2100 8650 2200
+Connection ~ 8650 2200
+$Comp
+L power:GND #PWR0107
+U 1 1 5E95B53A
+P 6100 3000
+F 0 "#PWR0107" H 6100 2750 50  0001 C CNN
+F 1 "GND" H 6105 2827 50  0000 C CNN
+F 2 "" H 6100 3000 50  0001 C CNN
+F 3 "" H 6100 3000 50  0001 C CNN
+	1    6100 3000
+	1    0    0    -1
+$EndComp
 $EndSCHEMATC
