File: powerBlock/powerBlock.sch (KiCad schematic (older format))
At the start: 30 parts, among them Q1 Q_PNP_EBC, Q2 Q_PNP_EBC, Q3 Q_PNP_EBC, U1 STM32F030C8Tx, U2 74HC164, U3 74HC164, U4 BA56-12SRWA

Commit message: Немного допилил схему. Немного оттрассировал
Parts:
- added C1, C10, C11: 10uF, Capacitor_SMD:C_0603_1608Metric, symbol Device:C
- added C2, C3: 100nF, Capacitor_SMD:C_0603_1608Metric, symbol Device:C
- added C4, C5, C6, C7, C8, C9: 1uF, Capacitor_SMD:C_0603_1608Metric, symbol Device:C
- added D10, D11, D12, D13, D9: DO-214AC, Diode_SMD:D_SMA, symbol pspice:DIODE
- added J2: Conn_01x10, Connector_PinHeader_2.54mm:PinHeader_1x10_P2.54mm_Horizontal, symbol Connector_Generic:Conn_01x10
- added J3: 282844-2, TerminalBlock_MetzConnect:TerminalBlock_MetzConnect_Type175_RT02702HBLC_1x02_P7.50mm_Horizontal, symbol Connector:Screw_Terminal_01x02
- added LS1: Speaker_Crystal, OptoDevice:R_LDR_10x8.5mm_P7.6mm_Vertical, symbol Device:Speaker_Crystal
- added Q4: BC857BMTF, Package_TO_SOT_SMD:SOT-23, symbol Device:Q_PNP_EBC
- added R16, R17, R19, R21, R23: 4.3kOhm, Resistor_SMD:R_0603_1608Metric, symbol Device:R
- added R18, R20, R22, R24: 470 Ohm, Resistor_SMD:R_0603_1608Metric, symbol Device:R
- added R25: 470Ohm, Resistor_SMD:R_0603_1608Metric, symbol Device:R
- added R26: 10kOhm, Resistor_SMD:R_0603_1608Metric, symbol Device:R
- added R27: 330 Ohm, Resistor_SMD:R_0603_1608Metric, symbol Device:R
- added RV1: TC33X-2-502E, Potentiometer_SMD:Potentiometer_Bourns_TC33X_Vertical, symbol Device:R_POT
- added SW1: SW_MEC_5G, Button_Switch_SMD:SW_SPST_PTS645, symbol Switch:SW_Push_Dual_x2
- added U5: LD1086DT50TR, Package_TO_SOT_SMD:TO-252-2, symbol Regulator_Linear:LD1086DT50TR
- added U6: AP2127K-3.3, Package_TO_SOT_SMD:SOT-23-5, symbol Regulator_Linear:AP2127K-3.3
- D1, D2, D3, D4, D5, D7, D8: footprint (none) -> LED_THT:LED_Rectangular_W3.9mm_H1.8mm
- J1: renamed from J?; footprint (none) -> Connector_PinHeader_2.54mm:PinHeader_1x04_P2.54mm_Vertical
- Q1, Q2, Q3: value Q_PNP_EBC -> BC857BMTF; footprint (none) -> Package_TO_SOT_SMD:SOT-23
- R1, R10, R11, R12, R13, R14, R15, R2, R3, R4, R5, R6, R7, R8, R9: footprint (none) -> Resistor_SMD:R_0603_1608Metric
Connections:
- net +5V: now also U2.14 (VCC), U2.9 (~MR), U3.9 (~MR)
- net GND: now also D1.1 (K), D2.1 (K), D3.1 (K), D4.1 (K), D5.1 (K), D7.1 (K), D8.1 (K), J1.4 (Pin_4), U1.23 (VSS), U1.47 (VSS), U1.8 (VSSA), U2.7 (GND), C10.2, C11.2, C2.2, C3.2, C4.2, C5.2, C6.2, C7.2, C8.2, C9.2, D10.1 (K), D11.1 (K), D12.1 (K), D13.1 (K), D9.1 (K), J3.2 (Pin_2), LS1.2, R18.1, R20.1, R22.1, R24.1, R25.1, RV1.1, SW1.2 (D), U5.1 (ADJ/GND), U6.2 (GND)
- net +3V3: now reaches U1.1 (VDD)
- net +3V3: now also J1.1 (Pin_1), U1.24 (VDD), U1.48 (VDD), U1.9 (VDDA), C2.1, C3.1, R26.1, U6.5 (VOUT)
- net ADC3: now reaches U1.13 (PA3)
- net ADC3: now also C4.1, D9.2 (A), R16.2, R25.2
- net ADC4: now reaches U1.14 (PA4)
- net ADC4: now also C5.1, D10.2 (A), R17.2, R18.2
- net ADC5: now reaches U1.15 (PA5)
- net ADC5: now also C6.1, D11.2 (A), R19.2, R20.2
- net ADC6: now reaches U1.16 (PA6)
- net ADC6: now also C7.1, D12.2 (A), R21.2, R22.2
- net ADC7: now reaches U1.17 (PA7)
- net ADC7: now also C8.1, D13.2 (A), R23.2, R24.2
- net at U1.32 (PA11): now also C9.1, R26.2, SW1.1 (C)
- net GPIOB8: now reaches U1.45 (PB8)
- net GPIOB8: now also Q4.2 (B)
- new net: LS1.1, RV1.2
- new net: R27.1, RV1.3
- new net: Q4.3 (C), R27.2
- new net +24АБ: J2.2 (Pin_2), R17.1
- new net +27В: J2.1 (Pin_1), R16.1
- new net +27В_СУ: C10.1, J3.1 (Pin_1), U5.3 (IN)
- new net +5VA: C1.1, C11.1, Q4.1 (E), U5.2 (OUT), U6.1 (VIN), U6.3 (EN)
- new net +U_vent: J2.3 (Pin_3), R19.1
- new net R_SH+: J2.4 (Pin_4), J2.6 (Pin_6), R23.1
- new net R_SH-: J2.5 (Pin_5), R21.1
- no-connect marks 1 -> 26
Other:
- note added: "1/(2*pi*R16*C)= F среза в герцах"
- moved on the sheet: J1
